File: esp32-4to20ma-board.kicad_sch (KiCad schematic)
At the start: 52 parts, among them J1 USB-C Receptacle, J2 4-20mA Loop, Q1 BCP53-16, Q2 MMBT5401, Q3 AO3401A, Q4 2N7002, SW1 RESET, SW2 BOOT, U1 ESP32-S3-WROOM-1U-N4, U3 INA226AIDGSR, U4 AP2112K-3.3, U5 MT3608

Commit message: Rev G: board routed, schematic regrouped, JLCPCB package
Routing
- route_board.py on routelib.py: the MT3608 loop (datasheet Figure 3), the
  INA226 Kelvin taps (Figure 30), the USB-C entry and pair, the power trunks,
  the 24 V loop, Q1's copper on both layers, every ground via and both pours
  are scripted; ten signal nets are Freerouting 2.4.1's, stored in
  routing/autoroute.json and replayed, so the board rebuilds byte-identically
  without Java. 0 unconnected, DRC unchanged at 4 + 5, parity clean, bottom
  ground in one piece, no via in any pad.
- Placement changes routing asked for: D1 turned 180 and moved up, R7/R8 into
  the lanes beside the connector, R10/R11 beside U5, C9 up 0.1 mm, R6/R15
  swapped so each pull-up sits under its own pin.
- setup_fab.py keeps the project's existing board rules (0.5 mm copper to edge).

Schematic
- Twelve hand-typed boxes became seven content-derived blocks, one per
  circuit, notes inside their block; nothing touches an outline (schlib's new
  outline check: ~100 faults on the old sheet, 0 now). Netlist unchanged:
  28 nets, ERC 0 errors. INA226 address pins share one ground port.
- Nine manufacturer names corrected against LCSC (every LCSC number and MPN
  was already right).

Fabrication
- build_package.py -> fab/: gerbers zip, 34-line BOM, 47-row CPL, order notes,
  behind a DRC gate. Standard PCBA is required (the ESP32-S3-WROOM-1U-N4 is
  "Standard Only" at JLCPCB). CPL rotations derived by jlc_compare.py from
  JLCPCB's own footprints: Q1-Q4 +180, everything else at zero; unverified
  until seen in their placement preview.

Housekeeping: the autorouter's work folder (scratch, with local paths in its
logs) was committed by mistake earlier; it is removed and ignored.

Co-Authored-By: Claude Fable 5.1 <noreply@anthropic.com>
Parts:
- C1, C6: Manufacturer Samwha/CCTC -> Samsung Electro-Mechanics
- C10, C11: Manufacturer Samsung/CCTC -> Samwha
- C12, C2, C3, C7, C8, C9: Manufacturer CCTC -> Samsung Electro-Mechanics
- D1: Manufacturer Ampec/ST-compatible -> UMW
- J1: Manufacturer Korean Hroparts Elec -> SHOU HAN
- L1: Manufacturer Sunlord -> cjiang
- LED1: Manufacturer Nichia-compatible -> Nationstar
- R10, R12, R21: Manufacturer Uniroyal -> FOJAN
- SW1, SW2: Manufacturer Korean Hroparts Elec -> Kinghelm
Other:
- note added: "+5V USB-C VBUS -> LDO, load switch +3V3 LDO -> ESP32-S3, INA226 +24V boost -> limiter -> loop terminal GND single ground plane"
- note added: "24 V BOOST CONVERTER - soft-start load switch, MT3608, feedback"
- note added: "3.3 V REGULATOR & POWER LED"
- note added: "ESP32-S3 MODULE - reset, boot, I2C pull-ups, decoupling"
- note added: "LOOP CURRENT LIMITER - 35 mA constant current, reverse blocking"
- note added: "LOOP TERMINAL & CURRENT MEASUREMENT - TVS, shunt, filter, INA226"
- note added: "POWER RAILS & SIGNAL LINKS"
- note added: "SIGNAL LINKS (net labels)"
- note added: "USB-C INPUT & ESD PROTECTION"
- note added: "USB_P / USB_N USB-C -> ESP32-S3 I2C_SDA / I2C_SCL ESP32-S3 -> INA226 MT_EN ESP32-S3 -> load switch LOOP_V / LOOP_RTN limiter -> terminal -> shunt"
- note removed: "+5V USB-C VBUS -> LDO, boost +3V3 LDO -> ESP32-S3, INA226 +24V boost -> loop terminal GND single ground plane"
- note removed: "24 V LOOP SUPPLY - MT3608 boost converter"
- note removed: "24 V OUTPUT & FEEDBACK"
- note removed: "3.3 V REGULATION"
- note removed: "4-20 mA LOOP - current limiter, shunt, input filter and INA226"
- note removed: "BOOST CONTROLLER"
- note removed: "BOOST INPUT"
- note removed: "CURRENT LIMITER"
- note removed: "ESP32-S3 MODULE"
- note removed: "INA226 CURRENT MONITOR"
- note removed: "LIMITER"
- note removed: "MICROCONTROLLER - ESP32-S3 module, reset and boot"
- note removed: "POWER INPUT - USB-C, ESD protection, 3.3 V regulation"
- note removed: "SECTION LINKS (net labels)"
- note removed: "SHUNT, FILTER & FIELD TERMINAL"
- note removed: "SOFT-START LOAD SWITCH"
- note removed: "STATUS"
- note removed: "SUPPORT CIRCUITRY"
- note removed: "USB-C INPUT & ESD"
- note removed: "USB_P / USB_N USB-C -> ESP32-S3 I2C_SDA / I2C_SCL ESP32-S3 -> INA226"
- moved on the sheet: C1, C10, C11, C12, C2, C3, C6, C7, C8, C9, D1, D2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
